Commit message: add RH56E2 Hand

File: urdf/AR5-5_07L-W4C4A2.urdf (robot description, URDF)
Before this commit: robot AR5-5_07L-W4C4A2, 10 links, 9 joints
Links:
- link AR5-5_07L-W4C4A2_base: geometry collision mesh filename=../meshes/AR5-5_07L-W4C4A2/AR5-5_07L-W4C4A2_base.stl scale=0.001 0.001 0.001; visual mesh filename=../meshes/AR5-5_07L-W4C4A2/AR5-5_07L-W4C4A2_base.stl scale=0.001 0.001 0.001
- link AR5-5_07L-W4C4A2_link1: geometry collision mesh filename=../meshes/AR5-5_07L-W4C4A2/AR5-5_07L-W4C4A2_link1.stl scale=0.001 0.001 0.001; visual mesh filename=../meshes/AR5-5_07L-W4C4A2/AR5-5_07L-W4C4A2_link1.stl scale=0.001 0.001 0.001
- link AR5-5_07L-W4C4A2_link2: geometry collision mesh filename=../meshes/AR5-5_07L-W4C4A2/AR5-5_07L-W4C4A2_link2.stl scale=0.001 0.001 0.001; visual mesh filename=../meshes/AR5-5_07L-W4C4A2/AR5-5_07L-W4C4A2_link2.stl scale=0.001 0.001 0.001
- link AR5-5_07L-W4C4A2_link3: geometry collision mesh filename=../meshes/AR5-5_07L-W4C4A2/AR5-5_07L-W4C4A2_link3.stl scale=0.001 0.001 0.001; visual mesh filename=../meshes/AR5-5_07L-W4C4A2/AR5-5_07L-W4C4A2_link3.stl scale=0.001 0.001 0.001
- link AR5-5_07L-W4C4A2_link4: geometry collision mesh filename=../meshes/AR5-5_07L-W4C4A2/AR5-5_07L-W4C4A2_link4.stl scale=0.001 0.001 0.001; visual mesh filename=../meshes/AR5-5_07L-W4C4A2/AR5-5_07L-W4C4A2_link4.stl scale=.001 0.001 0.001
- link AR5-5_07L-W4C4A2_link5: geometry collision mesh filename=../meshes/AR5-5_07L-W4C4A2/AR5-5_07L-W4C4A2_link5.stl scale=0.001 0.001 0.001; visual mesh filename=../meshes/AR5-5_07L-W4C4A2/AR5-5_07L-W4C4A2_link5.stl scale=0.001 0.001 0.001
- link AR5-5_07L-W4C4A2_link6: geometry collision mesh filename=../meshes/AR5-5_07L-W4C4A2/AR5-5_07L-W4C4A2_link6.stl scale=0.001 0.001 0.001; visual mesh filename=../meshes/AR5-5_07L-W4C4A2/AR5-5_07L-W4C4A2_link6.stl scale=0.001 0.001 0.001
- link AR5-5_07L-W4C4A2_link7: geometry collision mesh filename=../meshes/AR5-5_07L-W4C4A2/AR5-5_07L-W4C4A2_link7.stl scale=0.001 0.001 0.001; visual mesh filename=../meshes/AR5-5_07L-W4C4A2/AR5-5_07L-W4C4A2_link7.stl scale=0.001 0.001 0.001

File: urdf/AR5-5_07R-W4C4A2.urdf (robot description, URDF)
Before this commit: robot AR5-5_07R-W4C4A2, 10 links, 9 joints
Links:
- link AR5-5_07R-W4C4A2_base: geometry collision mesh filename=../meshes/AR5-5_07R-W4C4A2/AR5-5_07R-W4C4A2_base.stl scale=0.001 0.001 0.001; visual mesh filename=../meshes/AR5-5_07R-W4C4A2/AR5-5_07R-W4C4A2_base.stl scale=0.001 0.001 0.001
- link AR5-5_07R-W4C4A2_link1: geometry collision mesh filename=../meshes/AR5-5_07R-W4C4A2/AR5-5_07R-W4C4A2_link1.stl scale=0.001 0.001 0.001; visual mesh filename=../meshes/AR5-5_07R-W4C4A2/AR5-5_07R-W4C4A2_link1.stl scale=0.001 0.001 0.001
- link AR5-5_07R-W4C4A2_link2: geometry collision mesh filename=../meshes/AR5-5_07R-W4C4A2/AR5-5_07R-W4C4A2_link2.stl scale=0.001 0.001 0.001; visual mesh filename=../meshes/AR5-5_07R-W4C4A2/AR5-5_07R-W4C4A2_link2.stl scale=0.001 0.001 0.001
- link AR5-5_07R-W4C4A2_link3: geometry collision mesh filename=../meshes/AR5-5_07R-W4C4A2/AR5-5_07R-W4C4A2_link3.stl scale=0.001 0.001 0.001; visual mesh filename=../meshes/AR5-5_07R-W4C4A2/AR5-5_07R-W4C4A2_link3.stl scale=0.001 0.001 0.001
- link AR5-5_07R-W4C4A2_link4: geometry collision mesh filename=../meshes/AR5-5_07R-W4C4A2/AR5-5_07R-W4C4A2_link4.stl scale=0.001 0.001 0.001; visual mesh filename=../meshes/AR5-5_07R-W4C4A2/AR5-5_07R-W4C4A2_link4.stl scale=.001 0.001 0.001
- link AR5-5_07R-W4C4A2_link5: geometry collision mesh filename=../meshes/AR5-5_07R-W4C4A2/AR5-5_07R-W4C4A2_link5.stl scale=0.001 0.001 0.001; visual mesh filename=../meshes/AR5-5_07R-W4C4A2/AR5-5_07R-W4C4A2_link5.stl scale=0.001 0.001 0.001
- link AR5-5_07R-W4C4A2_link6: geometry collision mesh filename=../meshes/AR5-5_07R-W4C4A2/AR5-5_07R-W4C4A2_link6.stl scale=0.001 0.001 0.001; visual mesh filename=../meshes/AR5-5_07R-W4C4A2/AR5-5_07R-W4C4A2_link6.stl scale=0.001 0.001 0.001
- link AR5-5_07R-W4C4A2_link7: geometry collision mesh filename=../meshes/AR5-5_07R-W4C4A2/AR5-5_07R-W4C4A2_link7.stl scale=0.001 0.001 0.001; visual mesh filename=../meshes/AR5-5_07R-W4C4A2/AR5-5_07R-W4C4A2_link7.stl scale=0.001 0.001 0.001
