Commit message: update

File: AviatorRobot/bin/config/aviator_control.urdf (robot description, URDF)
Before this commit: robot aviator, 21 links, 20 joints
Joints:
- joint pitch_input_joint: limit lower=-0.165 upper=0 effort=10.0 velocity=1.0 -> lower=-0.170 upper=0 effort=10.0 velocity=1.0

File: AviatorRobot/bin/model/aviator_collision.urdf (robot description, URDF)
Before this commit: robot aviator_collision, 21 links, 20 joints
Joints:
- joint pitch_input_joint: limit lower=-0.165 upper=0 effort=10.0 velocity=1.0 -> lower=-0.170 upper=0 effort=10.0 velocity=1.0
