Commit message: update
profile	method	P50	P99	miss%	d_min	coll	e_task
sine	T0	0.78ms	1.59ms	0%	−15.5mm	8875	0.00
T4 (active)	34.6ms	38.2ms	100%	3.24mm	0	0.07
T5	0.069ms	0.085ms	0%	5.05mm	0	0.00
roll_pull	T0	0.75ms	1.57ms	0%	−15.3mm	8593	0.00
T5	0.072ms	0.087ms	0%	5.13mm	0	0.00
random	T0	0.79ms	2.34ms	0%	−17.7mm	8228	0.00
T4 (active)	39.1ms	76.8ms	100%	−17.7mm	7668	0.14
T5	0.070ms	0.096ms	0%	5.04mm	0	0.00

File: AviatorRobot/config/aviator_control.urdf (robot description, URDF)
Before this commit: robot aviator, 21 links, 20 joints
Joints:
- joint pitch_input_joint: limit lower=-0.170 upper=0 effort=10.0 velocity=1.0 -> lower=-0.165 upper=0 effort=10.0 velocity=1.0
