Commit message: fix: replace package:// URIs with relative paths in URDF
Change mesh references in aviator_collision.urdf from:
  package://aviator_meshes/aircraft_collision_0_ch.stl
to:
  meshes/aircraft_collision_0_ch.stl

This fixes the runtime error when loading collision meshes, as the
Pinocchio parser uses parentDir(urdf_path) as the package directory,
and the actual mesh files are located in the meshes/ subdirectory.

Fixes: Error: Mesh package://aviator_meshes/... could not be found

Co-Authored-By: Claude Opus 5.5 (1M context) <noreply@anthropic.com>

File: examples/AviatorRobot_simple/model/aviator_collision.urdf (robot description, URDF)
Before this commit: robot aviator_collision, 21 links, 20 joints
Links:
- link AR5-5_07L-W4C4A2_base: geometry collision mesh filename=meshes/AR5-5_07L-W4C4A2_base_ch.stl scale=1 1 1
- link AR5-5_07L-W4C4A2_link1: geometry collision mesh filename=meshes/AR5-5_07L-W4C4A2_link1_ch.stl scale=1 1 1
- link AR5-5_07L-W4C4A2_link2: geometry collision mesh filename=meshes/AR5-5_07L-W4C4A2_link2_ch.stl scale=1 1 1
- link AR5-5_07L-W4C4A2_link3: geometry collision mesh filename=meshes/AR5-5_07L-W4C4A2_link3_ch.stl scale=1 1 1
- link AR5-5_07L-W4C4A2_link4: geometry collision mesh filename=meshes/AR5-5_07L-W4C4A2_link4_ch.stl scale=1 1 1
- link AR5-5_07L-W4C4A2_link5: geometry collision mesh filename=meshes/AR5-5_07L-W4C4A2_link5_ch.stl scale=1 1 1
- link AR5-5_07L-W4C4A2_link6: geometry collision mesh filename=meshes/AR5-5_07L-W4C4A2_link6_ch.stl scale=1 1 1
- link AR5-5_07L-W4C4A2_link7: geometry collision mesh filename=meshes/AR5-5_07L-W4C4A2_link7_ch.stl scale=1 1 1
- link AR5-5_07R-W4C4A2_base: geometry collision mesh filename=meshes/AR5-5_07R-W4C4A2_base_ch.stl scale=1 1 1
- link AR5-5_07R-W4C4A2_link1: geometry collision mesh filename=meshes/AR5-5_07R-W4C4A2_link1_ch.stl scale=1 1 1
- link AR5-5_07R-W4C4A2_link2: geometry collision mesh filename=meshes/AR5-5_07R-W4C4A2_link2_ch.stl scale=1 1 1
- link AR5-5_07R-W4C4A2_link3: geometry collision mesh filename=meshes/AR5-5_07R-W4C4A2_link3_ch.stl scale=1 1 1
- link AR5-5_07R-W4C4A2_link4: geometry collision mesh filename=meshes/AR5-5_07R-W4C4A2_link4_ch.stl scale=1 1 1
- link AR5-5_07R-W4C4A2_link5: geometry collision mesh filename=meshes/AR5-5_07R-W4C4A2_link5_ch.stl scale=1 1 1
- link AR5-5_07R-W4C4A2_link6: geometry collision mesh filename=meshes/AR5-5_07R-W4C4A2_link6_ch.stl scale=1 1 1
- link AR5-5_07R-W4C4A2_link7: geometry collision mesh filename=meshes/AR5-5_07R-W4C4A2_link7_ch.stl scale=1 1 1
- link aircraft: geometry collision mesh filename=meshes/aircraft_collision_0_ch.stl scale=1 1 1; collision mesh filename=meshes/aircraft_collision_1_ch.stl scale=1 1 1
- link steering_wheel: geometry collision mesh filename=meshes/steering_wheel_collision_0_ch.stl scale=1 1 1; collision mesh filename=meshes/steering_wheel_collision_10_ch.stl scale=1 1 1
