Commit message: update

File: examples/AviatorRobot_simple/model/aviator_collision.urdf (robot description, URDF)
Before this commit: robot aviator_collision, 21 links, 20 joints
Joints:
- joint left_arm_base: origin xyz=-0.91333 0.008 0.12156 rpy=-1.5707 -0.1745329 0 -> xyz=-0.91333 0.010 0.12156 rpy=-1.5707 1.3962671  0
- joint right_arm_base: origin xyz=-0.91333 0.008 0.12156 rpy=1.5707 -0.1745329 0 -> xyz=-0.91333 -0.010 0.12156 rpy=1.5707 1.3962671  0
