Commit message: update

File: examples/AviatorRobot_simple/config/aviator_control.urdf (robot description, URDF)
Before this commit: robot aviator, 21 links, 20 joints
Joints:
- joint left_arm_base: origin xyz=-0.91333 0.008 0.12156 rpy=-1.5707 -0.1745329 0 -> xyz=-0.91333 0.008 0.12156 rpy=-1.5707 1.3962671  0
- joint right_arm_base: origin xyz=-0.91333 0.008 0.12156 rpy=1.5707 -0.1745329 0 -> xyz=-0.91333 -0.008 0.12156 rpy=1.5707 1.3962671  0

File: models/urdf/aviator.urdf (robot description, URDF)
Before this commit: robot aviator, 83 links, 82 joints
Joints:
- joint left_arm_base: origin xyz=-0.91333 0.008 0.12156 rpy=-1.5707 1.3962671 0 -> xyz=-0.91333 0.010 0.12156 rpy=-1.5707 1.3962671 0
- joint right_arm_base: origin xyz=-0.91333 0.008 0.12156 rpy=1.5707 1.3962671 0 -> xyz=-0.91333 -0.010 0.12156 rpy=1.5707 1.3962671 0

Commit message: update

File: examples/AviatorRobot_simple/config/aviator_control.urdf (robot description, URDF)
Before this commit: robot aviator, 21 links, 20 joints
Joints:
- joint left_arm_base: origin xyz=-0.91333 0.008 0.12156 rpy=-1.5707 1.3962671  0 -> xyz=-0.91333 0.010 0.12156 rpy=-1.5707 1.3962671  0
- joint right_arm_base: origin xyz=-0.91333 -0.008 0.12156 rpy=1.5707 1.3962671  0 -> xyz=-0.91333 -0.010 0.12156 rpy=1.5707 1.3962671  0
