Commit message: Reorganize model assets into urdf/meshes/mjcf directories
Move URDF/SRDF assets under models/urdf and meshes under models/meshes,
removing the duplicated models/control tree. Update robot.yaml, CMakeLists
install rules, docs, and tests to the new paths. Lower simulation
command/origin timeouts.

Co-Authored-By: Claude Code <noreply@anthropic.com>

File: models/urdf/aviator.urdf (robot description, URDF)
Before this commit: robot aviator, 83 links, 82 joints
Links:
- link aircraft: geometry collision mesh filename=../meshes/Cessna/aircraft.STL scale=1 1 1; visual mesh filename=../meshes/Cessna/aircraft.STL scale=1 1 1
- link steering_wheel: geometry collision mesh filename=../meshes/Cessna/steering_wheel.STL scale=1 1 1; visual mesh filename=../meshes/Cessna/steering_wheel.STL scale=1 1 1

File: models/urdf/aviator_collision.urdf (robot description, URDF)
Before this commit: robot aviator_collision, 21 links, 20 joints
Links:
- link AR5-5_07L-W4C4A2_base: geometry collision mesh filename=../meshes/AR5-5_07L-W4C4A2/AR5-5_07L-W4C4A2_base_ch.stl scale=1 1 1
- link AR5-5_07L-W4C4A2_link1: geometry collision mesh filename=../meshes/AR5-5_07L-W4C4A2/AR5-5_07L-W4C4A2_link1_ch.stl scale=1 1 1
- link AR5-5_07L-W4C4A2_link2: geometry collision mesh filename=../meshes/AR5-5_07L-W4C4A2/AR5-5_07L-W4C4A2_link2_ch.stl scale=1 1 1
- link AR5-5_07L-W4C4A2_link3: geometry collision mesh filename=../meshes/AR5-5_07L-W4C4A2/AR5-5_07L-W4C4A2_link3_ch.stl scale=1 1 1
- link AR5-5_07L-W4C4A2_link4: geometry collision mesh filename=../meshes/AR5-5_07L-W4C4A2/AR5-5_07L-W4C4A2_link4_ch.stl scale=1 1 1
- link AR5-5_07L-W4C4A2_link5: geometry collision mesh filename=../meshes/AR5-5_07L-W4C4A2/AR5-5_07L-W4C4A2_link5_ch.stl scale=1 1 1
- link AR5-5_07L-W4C4A2_link6: geometry collision mesh filename=../meshes/AR5-5_07L-W4C4A2/AR5-5_07L-W4C4A2_link6_ch.stl scale=1 1 1
- link AR5-5_07L-W4C4A2_link7: geometry collision mesh filename=../meshes/AR5-5_07L-W4C4A2/AR5-5_07L-W4C4A2_link7_ch.stl scale=1 1 1
- link AR5-5_07R-W4C4A2_base: geometry collision mesh filename=../meshes/AR5-5_07R-W4C4A2/AR5-5_07R-W4C4A2_base_ch.stl scale=1 1 1
- link AR5-5_07R-W4C4A2_link1: geometry collision mesh filename=../meshes/AR5-5_07R-W4C4A2/AR5-5_07R-W4C4A2_link1_ch.stl scale=1 1 1
- link AR5-5_07R-W4C4A2_link2: geometry collision mesh filename=../meshes/AR5-5_07R-W4C4A2/AR5-5_07R-W4C4A2_link2_ch.stl scale=1 1 1
- link AR5-5_07R-W4C4A2_link3: geometry collision mesh filename=../meshes/AR5-5_07R-W4C4A2/AR5-5_07R-W4C4A2_link3_ch.stl scale=1 1 1
- link AR5-5_07R-W4C4A2_link4: geometry collision mesh filename=../meshes/AR5-5_07R-W4C4A2/AR5-5_07R-W4C4A2_link4_ch.stl scale=1 1 1
- link AR5-5_07R-W4C4A2_link5: geometry collision mesh filename=../meshes/AR5-5_07R-W4C4A2/AR5-5_07R-W4C4A2_link5_ch.stl scale=1 1 1
- link AR5-5_07R-W4C4A2_link6: geometry collision mesh filename=../meshes/AR5-5_07R-W4C4A2/AR5-5_07R-W4C4A2_link6_ch.stl scale=1 1 1
- link AR5-5_07R-W4C4A2_link7: geometry collision mesh filename=../meshes/AR5-5_07R-W4C4A2/AR5-5_07R-W4C4A2_link7_ch.stl scale=1 1 1
- link aircraft: geometry collision mesh filename=../meshes/Cessna/aircraft_collision_0_ch.stl scale=1 1 1; collision mesh filename=../meshes/Cessna/aircraft_collision_1_ch.stl scale=1 1 1
- link steering_wheel: geometry collision mesh filename=../meshes/Cessna/steering_wheel_collision_0_ch.stl scale=1 1 1; collision mesh filename=../meshes/Cessna/steering_wheel_collision_10_ch.stl scale=1 1 1
