Commit message: update models

File: models/urdf/aviator.urdf (robot description, URDF)
Before this commit: robot aviator, 21 links, 20 joints
Links:
- added link l_base_link, mass 0.638115692832655; collision mesh filename=../meshes/RH56E2_L/l_base_link.STL; visual mesh filename=../meshes/RH56E2_L/l_base_link.STL
- added link left_index_1, mass 0.0182944233697246; collision mesh filename=../meshes/RH56E2_L/left_index_1.STL; visual mesh filename=../meshes/RH56E2_L/left_index_1.STL
- added link left_index_2, mass 0.0250395040688091; collision mesh filename=../meshes/RH56E2_L/left_index_2.STL; visual mesh filename=../meshes/RH56E2_L/left_index_2.STL
- added link left_index_force_sensor_1, mass 0.000202794475942539; collision mesh filename=../meshes/RH56E2_L/left_index_force_sensor_1.STL; visual mesh filename=../meshes/RH56E2_L/left_index_force_sensor_1.STL
- added link left_index_force_sensor_2, mass 0.000255748193489171; collision mesh filename=../meshes/RH56E2_L/left_index_force_sensor_2.STL; visual mesh filename=../meshes/RH56E2_L/left_index_force_sensor_2.STL
- added link left_index_force_sensor_3, mass 6.79653902597574E-05; collision mesh filename=../meshes/RH56E2_L/left_index_force_sensor_3.STL; visual mesh filename=../meshes/RH56E2_L/left_index_force_sensor_3.STL
- added link left_little_1, mass 0.0182944186286727; collision mesh filename=../meshes/RH56E2_L/left_little_1.STL; visual mesh filename=../meshes/RH56E2_L/left_little_1.STL
- added link left_little_2, mass 0.0193773130913926; collision mesh filename=../meshes/RH56E2_L/left_little_2.STL; visual mesh filename=../meshes/RH56E2_L/left_little_2.STL
- added link left_little_force_sensor_1, mass 0.000202794502264302; collision mesh filename=../meshes/RH56E2_L/left_little_force_sensor_1.STL; visual mesh filename=../meshes/RH56E2_L/left_little_force_sensor_1.STL
- added link left_little_force_sensor_2, mass 0.00028024674848609; collision mesh filename=../meshes/RH56E2_L/left_little_force_sensor_2.STL; visual mesh filename=../meshes/RH56E2_L/left_little_force_sensor_2.STL
- added link left_little_force_sensor_3, mass 6.10536670141796E-05; collision mesh filename=../meshes/RH56E2_L/left_little_force_sensor_3.STL; visual mesh filename=../meshes/RH56E2_L/left_little_force_sensor_3.STL
- added link left_middle_1, mass 0.0182944237783795; collision mesh filename=../meshes/RH56E2_L/left_middle_1.STL; visual mesh filename=../meshes/RH56E2_L/left_middle_1.STL
- added link left_middle_2, mass 0.027154082634411; collision mesh filename=../meshes/RH56E2_L/left_middle_2.STL; visual mesh filename=../meshes/RH56E2_L/left_middle_2.STL
- added link left_middle_force_sensor_1, mass 0.000202794522112893; collision mesh filename=../meshes/RH56E2_L/left_middle_force_sensor_1.STL; visual mesh filename=../meshes/RH56E2_L/left_middle_force_sensor_1.STL
- added link left_middle_force_sensor_2, mass 0.000262573593923136; collision mesh filename=../meshes/RH56E2_L/left_middle_force_sensor_2.STL; visual mesh filename=../meshes/RH56E2_L/left_middle_force_sensor_2.STL
- added link left_middle_force_sensor_3, mass 6.64914272946078E-05; collision mesh filename=../meshes/RH56E2_L/left_middle_force_sensor_3.STL; visual mesh filename=../meshes/RH56E2_L/left_middle_force_sensor_3.STL
- added link left_plam_casing, mass 0.0205046589058927; collision mesh filename=../meshes/RH56E2_L/left_plam_casing.STL; visual mesh filename=../meshes/RH56E2_L/left_plam_casing.STL
- added link left_plam_force_sensor, mass 0.00240886553361419; collision mesh filename=../meshes/RH56E2_L/left_plam_force_sensor.STL; visual mesh filename=../meshes/RH56E2_L/left_plam_force_sensor.STL
- added link left_ring_1, mass 0.018294421561901; collision mesh filename=../meshes/RH56E2_L/left_ring_1.STL; visual mesh filename=../meshes/RH56E2_L/left_ring_1.STL
- added link left_ring_2, mass 0.0250394550123085; collision mesh filename=../meshes/RH56E2_L/left_ring_2.STL; visual mesh filename=../meshes/RH56E2_L/left_ring_2.STL
- added link left_ring_force_sensor_1, mass 0.000202794434376475; collision mesh filename=../meshes/RH56E2_L/left_ring_force_sensor_1.STL; visual mesh filename=../meshes/RH56E2_L/left_ring_force_sensor_1.STL
- added link left_ring_force_sensor_2, mass 0.000255748190883573; collision mesh filename=../meshes/RH56E2_L/left_ring_force_sensor_2.STL; visual mesh filename=../meshes/RH56E2_L/left_ring_force_sensor_2.STL
- added link left_ring_force_sensor_3, mass 6.79657640763805E-05; collision mesh filename=../meshes/RH56E2_L/left_ring_force_sensor_3.STL; visual mesh filename=../meshes/RH56E2_L/left_ring_force_sensor_3.STL
- added link left_thumb_1, mass 0.00466740407248544; collision mesh filename=../meshes/RH56E2_L/left_thumb_1.STL; visual mesh filename=../meshes/RH56E2_L/left_thumb_1.STL
- added link left_thumb_2, mass 0.0385564917668049; collision mesh filename=../meshes/RH56E2_L/left_thumb_2.STL; visual mesh filename=../meshes/RH56E2_L/left_thumb_2.STL
- added link left_thumb_3, mass 0.0134342232166366; collision mesh filename=../meshes/RH56E2_L/left_thumb_3.STL; visual mesh filename=../meshes/RH56E2_L/left_thumb_3.STL
- added link left_thumb_4, mass 0.0226462079486484; collision mesh filename=../meshes/RH56E2_L/left_thumb_4.STL; visual mesh filename=../meshes/RH56E2_L/left_thumb_4.STL
- added link left_thumb_force_sensor_1, mass 0.000234351522411044; collision mesh filename=../meshes/RH56E2_L/left_thumb_force_sensor_1.STL; visual mesh filename=../meshes/RH56E2_L/left_thumb_force_sensor_1.STL
- added link left_thumb_force_sensor_2, mass 0.000119024235960818; collision mesh filename=../meshes/RH56E2_L/left_thumb_force_sensor_2.STL; visual mesh filename=../meshes/RH56E2_L/left_thumb_force_sensor_2.STL
- added link left_thumb_force_sensor_3, mass 0.000169894176021864; collision mesh filename=../meshes/RH56E2_L/left_thumb_force_sensor_3.STL; visual mesh filename=../meshes/RH56E2_L/left_thumb_force_sensor_3.STL
- added link left_thumb_force_sensor_4, mass 1.66991074236564E-05; collision mesh filename=../meshes/RH56E2_L/left_thumb_force_sensor_4.STL; visual mesh filename=../meshes/RH56E2_L/left_thumb_force_sensor_4.STL
- added link r_base_link, mass 0.640548028870977; collision mesh filename=../meshes/RH56E2_R/r_base_link.STL; visual mesh filename=../meshes/RH56E2_R/r_base_link.STL
- added link right_index_1, mass 0.0182957332404882; collision mesh filename=../meshes/RH56E2_R/right_index_1.STL; visual mesh filename=../meshes/RH56E2_R/right_index_1.STL
- added link right_index_2, mass 0.0250372341604781; collision mesh filename=../meshes/RH56E2_R/right_index_2.STL; visual mesh filename=../meshes/RH56E2_R/right_index_2.STL
- added link right_index_force_sensor_1, mass 0.00020277926206694; collision mesh filename=../meshes/RH56E2_R/right_index_force_sensor_1.STL; visual mesh filename=../meshes/RH56E2_R/right_index_force_sensor_1.STL
- added link right_index_force_sensor_2, mass 0.000255748458180208; collision mesh filename=../meshes/RH56E2_R/right_index_force_sensor_2.STL; visual mesh filename=../meshes/RH56E2_R/right_index_force_sensor_2.STL
- added link right_index_force_sensor_3, mass 6.79646984897729E-05; collision mesh filename=../meshes/RH56E2_R/right_index_force_sensor_3.STL; visual mesh filename=../meshes/RH56E2_R/right_index_force_sensor_3.STL
- added link right_little_1, mass 0.0182957029959314; collision mesh filename=../meshes/RH56E2_R/right_little_1.STL; visual mesh filename=../meshes/RH56E2_R/right_little_1.STL
- added link right_little_2, mass 0.00717697630300511; collision mesh filename=../meshes/RH56E2_R/right_little_2.STL; visual mesh filename=../meshes/RH56E2_R/right_little_2.STL
- added link right_little_force_sensor_1, mass 0.000202779290224811; collision mesh filename=../meshes/RH56E2_R/right_little_force_sensor_1.STL; visual mesh filename=../meshes/RH56E2_R/right_little_force_sensor_1.STL
- added link right_little_force_sensor_2, mass 0.000280265363825451; collision mesh filename=../meshes/RH56E2_R/right_little_force_sensor_2.STL; visual mesh filename=../meshes/RH56E2_R/right_little_force_sensor_2.STL
- added link right_little_force_sensor_3, mass 6.10539921684105E-05; collision mesh filename=../meshes/RH56E2_R/right_little_force_sensor_3.STL; visual mesh filename=../meshes/RH56E2_R/right_little_force_sensor_3.STL
- added link right_middle_1, mass 0.0182957332737578; collision mesh filename=../meshes/RH56E2_R/right_middle_1.STL; visual mesh filename=../meshes/RH56E2_R/right_middle_1.STL
- added link right_middle_2, mass 0.0271522531154338; collision mesh filename=../meshes/RH56E2_R/right_middle_2.STL; visual mesh filename=../meshes/RH56E2_R/right_middle_2.STL
- added link right_middle_force_sensor_1, mass 0.000202779388301744; collision mesh filename=../meshes/RH56E2_R/right_middle_force_sensor_1.STL; visual mesh filename=../meshes/RH56E2_R/right_middle_force_sensor_1.STL
- added link right_middle_force_sensor_2, mass 0.00026259331441686; collision mesh filename=../meshes/RH56E2_R/right_middle_force_sensor_2.STL; visual mesh filename=../meshes/RH56E2_R/right_middle_force_sensor_2.STL
- added link right_middle_force_sensor_3, mass 6.64914575467581E-05; collision mesh filename=../meshes/RH56E2_R/right_middle_force_sensor_3.STL; visual mesh filename=../meshes/RH56E2_R/right_middle_force_sensor_3.STL
- added link right_plam_casing, mass 0.0205048839956349; collision mesh filename=../meshes/RH56E2_R/right_plam_casing.STL; visual mesh filename=../meshes/RH56E2_R/right_plam_casing.STL
- added link right_plam_force_sensor, mass 0.00240887834862943; collision mesh filename=../meshes/RH56E2_R/right_plam_force_sensor.STL; visual mesh filename=../meshes/RH56E2_R/right_plam_force_sensor.STL
- added link right_ring_1, mass 0.0182957328723894; collision mesh filename=../meshes/RH56E2_R/right_ring_1.STL; visual mesh filename=../meshes/RH56E2_R/right_ring_1.STL
- added link right_ring_2, mass 0.0250372344903316; collision mesh filename=../meshes/RH56E2_R/right_ring_2.STL; visual mesh filename=../meshes/RH56E2_R/right_ring_2.STL
- added link right_ring_force_sensor_1, mass 0.00020277922338036; collision mesh filename=../meshes/RH56E2_R/right_ring_force_sensor_1.STL; visual mesh filename=../meshes/RH56E2_R/right_ring_force_sensor_1.STL
- added link right_ring_force_sensor_2, mass 0.000255748455642788; collision mesh filename=../meshes/RH56E2_R/right_ring_force_sensor_2.STL; visual mesh filename=../meshes/RH56E2_R/right_ring_force_sensor_2.STL
- added link right_ring_force_sensor_3, mass 6.79650392240318E-05; collision mesh filename=../meshes/RH56E2_R/right_ring_force_sensor_3.STL; visual mesh filename=../meshes/RH56E2_R/right_ring_force_sensor_3.STL
- added link right_thumb_1, mass 0.00466740407055572; collision mesh filename=../meshes/RH56E2_R/right_thumb_1.STL; visual mesh filename=../meshes/RH56E2_R/right_thumb_1.STL
- added link right_thumb_2, mass 0.0385554861475943; collision mesh filename=../meshes/RH56E2_R/right_thumb_2.STL; visual mesh filename=../meshes/RH56E2_R/right_thumb_2.STL
- added link right_thumb_3, mass 0.0134343727200358; collision mesh filename=../meshes/RH56E2_R/right_thumb_3.STL; visual mesh filename=../meshes/RH56E2_R/right_thumb_3.STL
- added link right_thumb_4, mass 0.0183095349526632; collision mesh filename=../meshes/RH56E2_R/right_thumb_4.STL; visual mesh filename=../meshes/RH56E2_R/right_thumb_4.STL
- added link right_thumb_force_sensor_1, mass 0.000234345870584151; collision mesh filename=../meshes/RH56E2_R/right_thumb_force_sensor_1.STL; visual mesh filename=../meshes/RH56E2_R/right_thumb_force_sensor_1.STL
- added link right_thumb_force_sensor_2, mass 0.000119024197892742; collision mesh filename=../meshes/RH56E2_R/right_thumb_force_sensor_2.STL; visual mesh filename=../meshes/RH56E2_R/right_thumb_force_sensor_2.STL
- added link right_thumb_force_sensor_3, mass 0.000169893832350008; collision mesh filename=../meshes/RH56E2_R/right_thumb_force_sensor_3.STL; visual mesh filename=../meshes/RH56E2_R/right_thumb_force_sensor_3.STL
- added link right_thumb_force_sensor_4, mass 1.66991205082656E-05; collision mesh filename=../meshes/RH56E2_R/right_thumb_force_sensor_4.STL; visual mesh filename=../meshes/RH56E2_R/right_thumb_force_sensor_4.STL
- link AR5-5_07L-W4C4A2_base: geometry collision mesh filename=../meshes/AR5-5_07L-W4C4A2/AR5-5_07L-W4C4A2_base.stl scale=0.001 0.001 0.001; visual mesh filename=../meshes/AR5-5_07L-W4C4A2/AR5-5_07L-W4C4A2_base.stl scale=0.001 0.001 0.001
- link AR5-5_07L-W4C4A2_link1: geometry collision mesh filename=../meshes/AR5-5_07L-W4C4A2/AR5-5_07L-W4C4A2_link1.stl scale=0.001 0.001 0.001; visual mesh filename=../meshes/AR5-5_07L-W4C4A2/AR5-5_07L-W4C4A2_link1.stl scale=0.001 0.001 0.001
- link AR5-5_07L-W4C4A2_link2: geometry collision mesh filename=../meshes/AR5-5_07L-W4C4A2/AR5-5_07L-W4C4A2_link2.stl scale=0.001 0.001 0.001; visual mesh filename=../meshes/AR5-5_07L-W4C4A2/AR5-5_07L-W4C4A2_link2.stl scale=0.001 0.001 0.001
- link AR5-5_07L-W4C4A2_link3: geometry collision mesh filename=../meshes/AR5-5_07L-W4C4A2/AR5-5_07L-W4C4A2_link3.stl scale=0.001 0.001 0.001; visual mesh filename=../meshes/AR5-5_07L-W4C4A2/AR5-5_07L-W4C4A2_link3.stl scale=0.001 0.001 0.001
- link AR5-5_07L-W4C4A2_link4: geometry collision mesh filename=../meshes/AR5-5_07L-W4C4A2/AR5-5_07L-W4C4A2_link4.stl scale=0.001 0.001 0.001; visual mesh filename=../meshes/AR5-5_07L-W4C4A2/AR5-5_07L-W4C4A2_link4.stl scale=.001 0.001 0.001
- link AR5-5_07L-W4C4A2_link5: geometry collision mesh filename=../meshes/AR5-5_07L-W4C4A2/AR5-5_07L-W4C4A2_link5.stl scale=0.001 0.001 0.001; visual mesh filename=../meshes/AR5-5_07L-W4C4A2/AR5-5_07L-W4C4A2_link5.stl scale=0.001 0.001 0.001
- link AR5-5_07L-W4C4A2_link6: geometry collision mesh filename=../meshes/AR5-5_07L-W4C4A2/AR5-5_07L-W4C4A2_link6.stl scale=0.001 0.001 0.001; visual mesh filename=../meshes/AR5-5_07L-W4C4A2/AR5-5_07L-W4C4A2_link6.stl scale=0.001 0.001 0.001
- link AR5-5_07L-W4C4A2_link7: geometry collision mesh filename=../meshes/AR5-5_07L-W4C4A2/AR5-5_07L-W4C4A2_link7.stl scale=0.001 0.001 0.001; visual mesh filename=../meshes/AR5-5_07L-W4C4A2/AR5-5_07L-W4C4A2_link7.stl scale=0.001 0.001 0.001
- link AR5-5_07R-W4C4A2_base: geometry collision mesh filename=../meshes/AR5-5_07R-W4C4A2/AR5-5_07R-W4C4A2_base.stl scale=0.001 0.001 0.001; visual mesh filename=../meshes/AR5-5_07R-W4C4A2/AR5-5_07R-W4C4A2_base.stl scale=0.001 0.001 0.001
- link AR5-5_07R-W4C4A2_link1: geometry collision mesh filename=../meshes/AR5-5_07R-W4C4A2/AR5-5_07R-W4C4A2_link1.stl scale=0.001 0.001 0.001; visual mesh filename=../meshes/AR5-5_07R-W4C4A2/AR5-5_07R-W4C4A2_link1.stl scale=0.001 0.001 0.001
- link AR5-5_07R-W4C4A2_link2: geometry collision mesh filename=../meshes/AR5-5_07R-W4C4A2/AR5-5_07R-W4C4A2_link2.stl scale=0.001 0.001 0.001; visual mesh filename=../meshes/AR5-5_07R-W4C4A2/AR5-5_07R-W4C4A2_link2.stl scale=0.001 0.001 0.001
- link AR5-5_07R-W4C4A2_link3: geometry collision mesh filename=../meshes/AR5-5_07R-W4C4A2/AR5-5_07R-W4C4A2_link3.stl scale=0.001 0.001 0.001; visual mesh filename=../meshes/AR5-5_07R-W4C4A2/AR5-5_07R-W4C4A2_link3.stl scale=0.001 0.001 0.001
- link AR5-5_07R-W4C4A2_link4: geometry collision mesh filename=../meshes/AR5-5_07R-W4C4A2/AR5-5_07R-W4C4A2_link4.stl scale=0.001 0.001 0.001; visual mesh filename=../meshes/AR5-5_07R-W4C4A2/AR5-5_07R-W4C4A2_link4.stl scale=.001 0.001 0.001
- link AR5-5_07R-W4C4A2_link5: geometry collision mesh filename=../meshes/AR5-5_07R-W4C4A2/AR5-5_07R-W4C4A2_link5.stl scale=0.001 0.001 0.001; visual mesh filename=../meshes/AR5-5_07R-W4C4A2/AR5-5_07R-W4C4A2_link5.stl scale=0.001 0.001 0.001
- link AR5-5_07R-W4C4A2_link6: geometry collision mesh filename=../meshes/AR5-5_07R-W4C4A2/AR5-5_07R-W4C4A2_link6.stl scale=0.001 0.001 0.001; visual mesh filename=../meshes/AR5-5_07R-W4C4A2/AR5-5_07R-W4C4A2_link6.stl scale=0.001 0.001 0.001
- link AR5-5_07R-W4C4A2_link7: geometry collision mesh filename=../meshes/AR5-5_07R-W4C4A2/AR5-5_07R-W4C4A2_link7.stl scale=0.001 0.001 0.001; visual mesh filename=../meshes/AR5-5_07R-W4C4A2/AR5-5_07R-W4C4A2_link7.stl scale=0.001 0.001 0.001
Joints:
- added joint RH56E2_L_joint: type fixed, parent AR5-5_07L-W4C4A2_flan_link, child l_base_link, origin xyz=0 0 -0.018 rpy=0 0 0
- added joint RH56E2_R_joint: type fixed, parent AR5-5_07R-W4C4A2_flan_link, child r_base_link, origin xyz=0 0 -0.018 rpy=0 0 0
- added joint left_index_1_joint: type revolute, parent l_base_link, child left_index_1, origin xyz=0.00056467 -0.038679 0.1564 rpy=1.6057 0 0, axis 0 0 -1, limit lower=0 upper=1.3700834628155487 effort=1 velocity=2
- added joint left_index_2_joint: type revolute, parent left_index_1, child left_index_2, origin xyz=0.0034259 0.032596 -0.00055 rpy=0 0 0, axis 0 0 -1, limit lower=0 upper=1.4855814987308995 effort=1 velocity=2, mimic joint=left_index_1_joint multiplier=1.0843 offset=0
- added joint left_index_force_sensor_1_joint: type fixed, parent left_index_1, child left_index_force_sensor_1, origin xyz=0.012046 0.019649 -0.006651 rpy=-1.5708 1.5351 -1.3587, axis 0 0 0
- added joint left_index_force_sensor_2_joint: type fixed, parent left_index_2, child left_index_force_sensor_2, origin xyz=0.0081655 0.037446 -0.0060795 rpy=-0.037141 0 -0.34877, axis 0 0 0
- added joint left_index_force_sensor_3_joint: type fixed, parent left_index_2, child left_index_force_sensor_3, origin xyz=0.0086237 0.052572 -0.0060954 rpy=-1.5708 1.5252 -0.87237, axis 0 0 0
- added joint left_little_1_joint: type revolute, parent l_base_link, child left_little_1, origin xyz=0.000564666676608427 0.025916086514562 0.153652298734666 rpy=1.46607657167525 0 0, axis 0 0 -1, limit lower=0 upper=1.3700834628155487 effort=1 velocity=2
- added joint left_little_2_joint: type revolute, parent left_little_1, child left_little_2, origin xyz=0.0034259 0.032596 -0.00055 rpy=0 0 0, axis 0 0 -1, limit lower=0 upper=1.4855814987308995 effort=1 velocity=2, mimic joint=left_little_1_joint multiplier=1.0843 offset=0
- added joint left_little_force_sensor_1_joint: type fixed, parent left_little_1, child left_little_force_sensor_1, origin xyz=0.012046 0.019649 -0.006651 rpy=1.5708 1.4637 1.7829, axis 0 0 0
- added joint left_little_force_sensor_2_joint: type fixed, parent left_little_2, child left_little_force_sensor_2, origin xyz=0.00645136106946357 0.0276831973860534 -0.00611719269601713 rpy=1.57079632679489 1.45969392220978 1.22888814143765, axis 0 0 0
- added joint left_little_force_sensor_3_joint: type fixed, parent left_little_2, child left_little_force_sensor_3, origin xyz=0.00639726945590022 0.0427069119558453 -0.00611540980074188 rpy=1.5707963267949 1.43362674619756 2.27608569263426, axis 0 0 0
- added joint left_middle_1_joint: type revolute, parent l_base_link, child left_middle_1, origin xyz=0.00056467 -0.0171 0.157 rpy=1.5708 0 0, axis 0 0 -1, limit lower=0 upper=1.3700834628155487 effort=1 velocity=2
- added joint left_middle_2_joint: type revolute, parent left_middle_1, child left_middle_2, origin xyz=0.0034259 0.032596 -0.00055 rpy=0 0 0, axis 0 0 -1, limit lower=0 upper=1.4855814987308995 effort=1 velocity=2, mimic joint=left_middle_1_joint multiplier=1.0843 offset=0
- added joint left_middle_force_sensor_1_joint: type fixed, parent left_middle_1, child left_middle_force_sensor_1, origin xyz=0.012046 0.019649 -0.006651 rpy=-1.6995 1.5708 -1.4874, axis 0 0 0
- added joint left_middle_force_sensor_2_joint: type fixed, parent left_middle_2, child left_middle_force_sensor_2, origin xyz=0.009086 0.040962 -0.0061003 rpy=0.12266 1.5708 -0.25019, axis 0 0 0
- added joint left_middle_force_sensor_3_joint: type fixed, parent left_middle_2, child left_middle_force_sensor_3, origin xyz=0.0098294 0.056051 -0.0061006 rpy=-0.67435 1.5708 0, axis 0 0 0
- added joint left_plam_casing_joint: type fixed, parent l_base_link, child left_plam_casing, origin xyz=0 0 0.031 rpy=0 0 0, axis 0 0 0
- added joint left_plam_force_sensor_joint: type fixed, parent l_base_link, child left_plam_force_sensor, origin xyz=0.0122962567472441 -0.000368185252603959 0.119601267398173 rpy=1.57079632679489 0 1.5707963267949, axis 0 0 0
- added joint left_ring_1_joint: type revolute, parent l_base_link, child left_ring_1, origin xyz=0.00056467 0.0045302 0.15683 rpy=1.5184 0 0, axis 0 0 -1, limit lower=0 upper=1.3700834628155487 effort=1 velocity=2
- added joint left_ring_2_joint: type revolute, parent left_ring_1, child left_ring_2, origin xyz=0.0034259 0.032596 -0.00055 rpy=0 0 0, axis 0 0 -1, limit lower=0 upper=1.4855814987308995 effort=1 velocity=2, mimic joint=left_ring_1_joint multiplier=1.0843 offset=0
- added joint left_ring_force_sensor_1_joint: type fixed, parent left_ring_1, child left_ring_force_sensor_1, origin xyz=0.012046 0.019649 -0.006651 rpy=1.5708 1.5172 1.7829, axis 0 0 0
- added joint left_ring_force_sensor_2_joint: type fixed, parent left_ring_2, child left_ring_force_sensor_2, origin xyz=0.0081655 0.037446 -0.0060795 rpy=1.5708 1.5151 1.222, axis 0 0 0
- added joint left_ring_force_sensor_3_joint: type fixed, parent left_ring_2, child left_ring_force_sensor_3, origin xyz=0.0086237 0.052572 -0.0060954 rpy=1.5708 1.5025 2.2692, axis 0 0 0
- added joint left_thumb_1_joint: type revolute, parent l_base_link, child left_thumb_1, origin xyz=0.02101 -0.0269 0.0826 rpy=0 0 0, axis 0 0 1, limit lower=0 upper=1.6580627893946132 effort=1 velocity=2
- added joint left_thumb_2_joint: type revolute, parent left_thumb_1, child left_thumb_2, origin xyz=0.013438 -0.012862 -0.0076 rpy=1.5708 0 -1.5708, axis 0.17365 0 0.98481, limit lower=0 upper=0.6195918844579870 effort=1 velocity=2
- added joint left_thumb_3_joint: type revolute, parent left_thumb_2, child left_thumb_3, origin xyz=0.052954 0.032799 -0.0093372 rpy=0 0 0, axis 0.17365 0 0.98481, limit lower=0 upper=0.5199615094371426 effort=1 velocity=2, mimic joint=left_thumb_2_joint multiplier=0.8392 offset=0
- added joint left_thumb_4_joint: type revolute, parent left_thumb_3, child left_thumb_4, origin xyz=0.01865 0.013373 -0.0022731 rpy=0 0 0, axis 0.17365 0 0.98481, limit lower=0 upper=0.4632857049084941 effort=1 velocity=2, mimic joint=left_thumb_3_joint multiplier=0.891 offset=0
- added joint left_thumb_force_sensor_1_joint: type fixed, parent left_thumb_2, child left_thumb_force_sensor_1, origin xyz=0.023412 0.033251 0.0070079 rpy=1.1285 1.3976 3.1383, axis 0 0 0
- added joint left_thumb_force_sensor_2_joint: type fixed, parent left_thumb_3, child left_thumb_force_sensor_2, origin xyz=0.0080283 0.016443 0.00982 rpy=0.96257 1.4071 3.0993, axis 0 0 0
- added joint left_thumb_force_sensor_3_joint: type fixed, parent left_thumb_4, child left_thumb_force_sensor_3, origin xyz=0.0076349 0.020486 0.0088094 rpy=0.64092 1.3963 -3.1415, axis 0 0 0
- added joint left_thumb_force_sensor_4_joint: type fixed, parent left_thumb_4, child left_thumb_force_sensor_4, origin xyz=0.018831 0.027914 0.0068352 rpy=1.7521 1.3962 -3.1401, axis 0 0 0
- added joint right_index_1_joint: type revolute, parent r_base_link, child right_index_1, origin xyz=0.00056467 0.038679 0.1564 rpy=1.5359 0 0, axis 0 0 -1, limit lower=0 upper=1.3700834628155487 effort=1 velocity=1
- added joint right_index_2_joint: type revolute, parent right_index_1, child right_index_2, origin xyz=0.0034259 0.032596 0.00055 rpy=0 0 0, axis 0 0 -1, limit lower=0 upper=1.4855814987308995 effort=1 velocity=1, mimic joint=right_index_1_joint multiplier=1.0843 offset=0
- added joint right_index_force_sensor_1_joint: type fixed, parent right_index_1, child right_index_force_sensor_1, origin xyz=0.012046 0.019649 0.006651 rpy=1.5708 1.5351 1.7829, axis 0 0 0
- added joint right_index_force_sensor_2_joint: type fixed, parent right_index_2, child right_index_force_sensor_2, origin xyz=0.0081655 0.037446 0.0060795 rpy=1.5708 1.5337 1.222, axis 0 0 0
- added joint right_index_force_sensor_3_joint: type fixed, parent right_index_2, child right_index_force_sensor_3, origin xyz=0.0086237 0.052572 0.0060954 rpy=1.5708 1.5252 2.2692, axis 0 0 0
- added joint right_little_1_joint: type revolute, parent r_base_link, child right_little_1, origin xyz=0.00056467 -0.025916 0.15365 rpy=1.6755 0 0, axis 0 0 -1, limit lower=0 upper=1.3700834628155487 effort=1 velocity=1
- added joint right_little_2_joint: type revolute, parent right_little_1, child right_little_2, origin xyz=0.0034259 0.032596 0.00055 rpy=0 0 0, axis 0 0 -1, limit lower=0 upper=1.4855814987308995 effort=1 velocity=1, mimic joint=right_little_1_joint multiplier=1.0843 offset=0
- added joint right_little_force_sensor_1_joint: type fixed, parent right_little_1, child right_little_force_sensor_1, origin xyz=0.012046 0.019649 0.006651 rpy=-1.5708 1.4637 -1.3587, axis 0 0 0
- added joint right_little_force_sensor_2_joint: type fixed, parent right_little_2, child right_little_force_sensor_2, origin xyz=0.0064512 0.027683 0.0061172 rpy=-1.5708 1.4597 -1.9127, axis 0 0 0
- added joint right_little_force_sensor_3_joint: type fixed, parent right_little_2, child right_little_force_sensor_3, origin xyz=0.0063972 0.042707 0.0061154 rpy=-1.5708 1.4336 -0.86551, axis 0 0 0
- added joint right_middle_1_joint: type revolute, parent r_base_link, child right_middle_1, origin xyz=0.00056467 0.0171 0.157 rpy=1.5708 0 0, axis 0 0 -1, limit lower=0 upper=1.3700834628155487 effort=1 velocity=1
- added joint right_middle_2_joint: type revolute, parent right_middle_1, child right_middle_2, origin xyz=0.0034259 0.032596 0.00055 rpy=0 0 0, axis 0 0 -1, limit lower=0 upper=1.4855814987308995 effort=1 velocity=1, mimic joint=right_middle_1_joint multiplier=1.0843 offset=0
- added joint right_middle_force_sensor_1_joint: type fixed, parent right_middle_1, child right_middle_force_sensor_1, origin xyz=0.012046 0.019649 0.006651 rpy=-0.21209 1.5708 0, axis 0 0 0
- added joint right_middle_force_sensor_2_joint: type fixed, parent right_middle_2, child right_middle_force_sensor_2, origin xyz=0.0090859 0.040963 0.0061003 rpy=0.37285 1.5708 0, axis 0 0 0
- added joint right_middle_force_sensor_3_joint: type fixed, parent right_middle_2, child right_middle_force_sensor_3, origin xyz=0.0098294 0.056051 0.0061006 rpy=-0.67435 1.5708 0, axis 0 0 0
- added joint right_plam_casing_joint: type fixed, parent r_base_link, child right_plam_casing, origin xyz=0 0 0.030747 rpy=0 0 0, axis 0 0 0
- added joint right_plam_force_sensor_joint: type fixed, parent r_base_link, child right_plam_force_sensor, origin xyz=0.012296 0.00036819 0.1196 rpy=1.5708 0 1.5708, axis 0 0 0
- added joint right_ring_1_joint: type revolute, parent r_base_link, child right_ring_1, origin xyz=0.00056467 -0.0045302 0.15683 rpy=1.6232 0 0, axis 0 0 -1, limit lower=0 upper=1.3700834628155487 effort=1 velocity=1
- added joint right_ring_2_joint: type revolute, parent right_ring_1, child right_ring_2, origin xyz=0.0034259 0.032596 0.00055 rpy=0 0 0, axis 0 0 -1, limit lower=0 upper=1.4855814987308995 effort=1 velocity=1, mimic joint=right_ring_1_joint multiplier=1.0843 offset=0
- added joint right_ring_force_sensor_1_joint: type fixed, parent right_ring_1, child right_ring_force_sensor_1, origin xyz=0.012046 0.019649 0.006651 rpy=-1.5708 1.5172 -1.3587, axis 0 0 0
- added joint right_ring_force_sensor_2_joint: type fixed, parent right_ring_2, child right_ring_force_sensor_2, origin xyz=0.0081655 0.037446 0.0060795 rpy=-1.5708 1.5151 -1.9196, axis 0 0 0
- added joint right_ring_force_sensor_3_joint: type fixed, parent right_ring_2, child right_ring_force_sensor_3, origin xyz=0.0086237 0.052572 0.0060954 rpy=-1.5708 1.5025 -0.87237, axis 0 0 0
- added joint right_thumb_1_joint: type revolute, parent r_base_link, child right_thumb_1, origin xyz=0.02101 0.0269 0.0826 rpy=0 0 0, axis 0 0 -1, limit lower=0 upper=1.6580627893946132 effort=1 velocity=2
- added joint right_thumb_2_joint: type revolute, parent right_thumb_1, child right_thumb_2, origin xyz=0.013438 0.012862 -0.0076 rpy=1.5708 0 -1.5708, axis 0.17365 0 -0.98481, limit lower=0 upper=0.6195918844579870 effort=1 velocity=2
- added joint right_thumb_3_joint: type revolute, parent right_thumb_2, child right_thumb_3, origin xyz=-0.052954 0.032799 -0.0093372 rpy=0 0 0, axis 0.17365 0 -0.98481, limit lower=0 upper=0.5199615094371426 effort=1 velocity=2, mimic joint=right_thumb_2_joint multiplier=0.8392 offset=0
- added joint right_thumb_4_joint: type revolute, parent right_thumb_3, child right_thumb_4, origin xyz=-0.01865 0.013373 -0.0022731 rpy=0 0 0, axis 0.17365 0 -0.98481, limit lower=0 upper=0.4632857049084941 effort=1 velocity=2, mimic joint=right_thumb_3_joint multiplier=0.891 offset=0
- added joint right_thumb_force_sensor_1_joint: type fixed, parent right_thumb_2, child right_thumb_force_sensor_1, origin xyz=-0.023424 0.033251 0.007073 rpy=-0.99905 1.4338 0.13409, axis 0 0 0
- added joint right_thumb_force_sensor_2_joint: type fixed, parent right_thumb_3, child right_thumb_force_sensor_2, origin xyz=-0.0080057 0.016443 0.0096921 rpy=-1.041 1.3851 -0.037357, axis 0 0 0
- added joint right_thumb_force_sensor_3_joint: type fixed, parent right_thumb_4, child right_thumb_force_sensor_3, origin xyz=-0.0076345 0.020486 0.0088067 rpy=-0.64083 1.3963 4.2914E-05, axis 0 0 0
- added joint right_thumb_force_sensor_4_joint: type fixed, parent right_thumb_4, child right_thumb_force_sensor_4, origin xyz=-0.01883 0.027914 0.0068326 rpy=-1.7492 1.3963 0.0014317, axis 0 0 0
- joint pitch_input_joint: limit lower=-0.170 upper=0 effort=10.0 velocity=1.0 -> lower=-0.165 upper=0 effort=10.0 velocity=1.0
