Commit message: Enhances build, node startup, and robot model accuracy
* Introduces a `aviator_add_test_executable` CMake function to consolidate all test binaries into a dedicated `build/tests` directory, separating them from application executables.
* Improves third-party dependency management by propagating MuJoCo include paths and refining build order for robotics libraries (Pinocchio, PIN-IK, Coal). Missing third-party sources now result in a fatal error during configuration.
* Adds structured startup information panels for core nodes (`aviator_bus`, `aviator_monitor`, `flight_gateway`, `simulation`). These panels provide immediate operational details like endpoints, topics, and status, improving user experience and debugging.
* Corrects the orientation of the robot's hands in the URDF and MJCF models, improving the physical accuracy of the simulation.
* Updates the default bus endpoints for the simulation node to align with the main application bus (5555/5556), simplifying integration.

File: models/urdf/aviator.urdf (robot description, URDF)
Before this commit: robot aviator, 83 links, 82 joints
Joints:
- joint RH56E2_L_joint: origin xyz=0 0 -0.018 rpy=0 0 0 -> xyz=0 0 -0.018 rpy=0 0 1.5708
- joint RH56E2_R_joint: origin xyz=0 0 -0.018 rpy=0 0 0 -> xyz=0 0 -0.018 rpy=0 0 -1.5708

Commit message: Update models

File: models/urdf/aviator.urdf (robot description, URDF)
Before this commit: robot aviator, 83 links, 82 joints
Joints:
- joint left_arm_base: origin xyz=-0.91333 0.008 0.12156 rpy=-1.5707 -0.1745329 0 -> xyz=-0.91333 0.008 0.12156 rpy=-1.5707 1.3962671 0
- joint right_arm_base: origin xyz=-0.91333 0.008 0.12156 rpy=1.5707 -0.1745329 0 -> xyz=-0.91333 0.008 0.12156 rpy=1.5707 1.3962671 0

Commit message: update model

File: models/urdf/aviator.urdf (robot description, URDF)
Before this commit: robot aviator, 83 links, 82 joints
Links:
- link aircraft: geometry collision mesh filename=../meshes/aircraft.STL scale=1 1 1; visual mesh filename=../meshes/aircraft.STL scale=1 1 1
Joints:
- joint left_arm_base: origin xyz=-0.91333 0.010 0.12156 rpy=-1.5707 1.3962671 0 -> xyz=-0.91333 0.010 0.12156 rpy=-1.5707 1.5708 0
- joint right_arm_base: origin xyz=-0.91333 -0.010 0.12156 rpy=1.5707 1.3962671 0 -> xyz=-0.91333 -0.010 0.12156 rpy=1.5707 1.5708 0

Commit message: update models

File: models/urdf/aviator.urdf (robot description, URDF)
Before this commit: robot aviator, 83 links, 82 joints
Joints:
- joint RH56E2_L_joint: origin xyz=0 0 -0.018 rpy=0 0 1.5708 -> xyz=0 0 0.0116 rpy=0 0 1.5708
- joint RH56E2_R_joint: origin xyz=0 0 -0.018 rpy=0 0 -1.5708 -> xyz=0 0 0.0116 rpy=0 0 -1.5708

Commit message: update urdf

File: models/urdf/aviator.urdf (robot description, URDF)
Before this commit: robot aviator, 83 links, 82 joints
Links:
- added link dummy_link_2
- added link shell; visual mesh filename=../meshes/Cessna/shell.STL scale=1 1 1
- added link steering_wheel_2, mass 0.5; visual mesh filename=../meshes/Cessna/steering_wheel_2.STL scale=1 1 1
- link aircraft: geometry visual mesh filename=../meshes/Cessna/aircraft_visual.STL scale=1 1 1
- link steering_wheel: geometry collision mesh filename=../meshes/Cessna/steering_wheel_qr.STL scale=1 1 1; visual mesh filename=../meshes/Cessna/steering_wheel_qr.STL scale=1 1 1
Joints:
- added joint fixed_shell: type fixed, parent aircraft, child shell, origin xyz=0 0 0 rpy=0 0 0
- added joint pitch_input_joint_2: type prismatic, parent dummy_link_2, child steering_wheel_2, origin xyz=0 0 0 rpy=0 0 0, axis 0 0 1, limit lower=-0.170 upper=0 effort=10.0 velocity=1.0, mimic joint=pitch_input_joint multiplier=1.0
- added joint roll_input_joint_2: type revolute, parent aircraft, child dummy_link_2, origin xyz=0 0.47 0 rpy=1.5707 0 -1.5707, axis 0 0 1, limit lower=-0.87266 upper=0.87266 effort=10.0 velocity=1.0, mimic joint=roll_input_joint multiplier=1.0

Commit message: update

File: models/urdf/aviator.urdf (robot description, URDF)
Before this commit: robot aviator, 86 links, 85 joints
Links:
- link steering_wheel: geometry collision mesh filename=../meshes/Cessna/narrow/steering_wheel_qr.STL scale=1 1 1; visual mesh filename=../meshes/Cessna/narrow/steering_wheel_qr.STL scale=1 1 1
Joints:
- joint left_arm_base: origin xyz=-0.91333 0.010 0.12156 rpy=-1.5707 1.5708 0 -> xyz=-0.91333 0.020 0.13756 rpy=-1.5707 1.5708 0
- joint right_arm_base: origin xyz=-0.91333 -0.010 0.12156 rpy=1.5707 1.5708 0 -> xyz=-0.91333 0.000 0.13756 rpy=1.5707 1.5708 0
